File: hardware-design/kicad/dilder-breadboard/dilder-breadboard.kicad_sch (KiCad schematic)
At the start: 0 parts

Commit message: Fix KiCad schematic — remove invalid comment syntax, fix project UUID
Removed ;; comment lines that KiCad's S-expression parser cannot handle.
Fixed malformed UUID in project sheets reference. Schematic now loads
cleanly in KiCad 8+.

Co-Authored-By: Claude Opus 4.6 (1M context) <noreply@anthropic.com>
Other:
- note added: "1. HC-SR04 ECHO is 5V output — MUST use voltage divider or damage Pico"
- note added: "2. GPS TX/RX crossover: GPS TX goes to Pico RX, GPS RX to Pico TX"
- note added: "3. Joystick uses Pico internal pull-ups — no external resistors"
- note added: "3V3 --> Speaker(+) --> Speaker(-) --> NPN Collector"
- note added: "3V3 [Pin 36] — e-Paper VCC + GPS VCC (3.3V power)"
- note added: "4. Speaker: piezo direct to GP15+GND, or NPN transistor for volume"
- note added: "5. Total GPIO used: 16 of 26 — 10 pins free for future sensors"
- note added: "6. 3V3 rail max 300mA — all peripherals draw about 120mA total"
- note added: "BUSY ----> GP13 [Pin 17]"
- note added: "CENTER ----> GP6 [Pin 9]"
- note added: "CLK ----> GP10 SPI1 SCK [Pin 14]"
- note added: "COM/GND ----> GND [Pin 8]"
- note added: "CS ----> GP9 SPI1 CSn [Pin 12]"
- note added: "DC ----> GP8 [Pin 11]"
- note added: "DIN ----> GP11 SPI1 TX [Pin 15]"
- note added: "DOWN ----> GP3 [Pin 5]"
- note added: "E-PAPER DISPLAY — Waveshare 2.13 inch V3 (SPI1, 4MHz)"
- note added: "GND ----> GND [Pin 38]"
- note added: "GND --> NPN Emitter"
- note added: "GND [Pin 13]"
- note added: "GND [Pin 18]"
- note added: "GND [Pin 23] — HC-SR04 GND + Speaker GND"
- note added: "GND [Pin 28]"
- note added: "GND [Pin 38] — e-Paper GND"
- note added: "GND [Pin 3] — GPS GND"
- note added: "GND [Pin 8] — Joystick COM / GND"
- note added: "GP0 [Pin 1] — UART0 TX --> GPS RX"
- note added: "GP1 [Pin 2] — UART0 RX <-- GPS TX"
- note added: "GP10 [Pin 14] — e-Paper CLK (SPI1 SCK)"
- note added: "GP11 [Pin 15] — e-Paper DIN (SPI1 TX / MOSI)"
- note added: "GP12 [Pin 16] — e-Paper RST"
- note added: "GP13 [Pin 17] — e-Paper BUSY"
- note added: "GP14 [Pin 19] — HC-SR04 TRIG (output)"
- note added: "GP15 [Pin 20] — Speaker PWM (output)"
- note added: "GP16 [Pin 21] — HC-SR04 ECHO (via voltage divider)"
- note added: "GP2 [Pin 4] — Joystick UP (pull-up, active LOW)"
- note added: "GP3 [Pin 5] — Joystick DOWN"
- note added: "GP4 [Pin 6] — Joystick LEFT"
- note added: "GP5 [Pin 7] — Joystick RIGHT"
- note added: "GP6 [Pin 9] — Joystick CENTER / SELECT"
- note added: "GP7 [Pin 10] — FREE"
- note added: "GP8 [Pin 11] — e-Paper DC"
- note added: "GP9 [Pin 12] — e-Paper CS (SPI1 CSn)"
- note added: "GPS GND ----> GND [Pin 3]"
- note added: "GPS MODULE — GY-NEO6MV2 (UART0, 9600 baud)"
- note added: "GPS RX <---- Pico GP0 (UART0 TX) [Pin 1] << TX-RX CROSSOVER"
- note added: "GPS TX ----> Pico GP1 (UART0 RX) [Pin 2] << TX-RX CROSSOVER"
- note added: "GPS VCC ----> 3V3(OUT) [Pin 36]"
- note added: "HC-SR04 ECHO VOLTAGE DIVIDER (5V to 3.3V) — REQUIRED"
- note added: "HC-SR04 ECHO pin ---[ 1K ohm R1 ]---+--- GP16 (Pin 21)"
- note added: "JOYSTICK — DollaTek 5-Way (Active LOW, Internal Pull-ups)"
- note added: "LEFT ----> GP4 [Pin 6]"
- note added: "LEFT SIDE"
- note added: "NPN transistor: 2N2222, BC547, or BC817"
- note added: "Option A (simple): GP15 ----> Piezo(+) Piezo(-) ----> GND"
- note added: "Option B (louder): GP15 --[ 1K R3 ]--> NPN Base"
- note added: "RASPBERRY PI PICO WH — PIN ASSIGNMENTS"
- note added: "RIGHT ----> GP5 [Pin 7]"
- note added: "RIGHT SIDE"
- note added: "RST ----> GP12 [Pin 16]"
- note added: "SPEAKER CIRCUIT (GP15 PWM)"
- note added: "UP ----> GP2 [Pin 4]"
- note added: "VBUS [Pin 40] — HC-SR04 VCC (5V)"
- note added: "VCC ----> 3V3(OUT) [Pin 36]"
- note added: "VSYS [Pin 39] — (Battery future)"
- note added: "Vout = 5V x 2K / (1K + 2K) = 3.33V -- Safe for Pico 3.3V GPIO"
- note added: "[ 2K ohm R2 ]"
- note added: "|"
- note removed: "1. HC-SR04 ECHO is 5V — MUST use voltage divider (1KΩ + 2KΩ) or damage Pico"
- note removed: "2. GPS TX→RX crossover: GPS TX connects to Pico RX (GP1), GPS RX to Pico TX (GP0)"
- note removed: "3. All joystick directions use Pico internal pull-ups — no external resistors needed"
- note removed: "3V3 [36] — e-Paper VCC + GPS VCC"
- note removed: "3V3 ──→ Speaker(+) ──→ Speaker(-) ──→ Collector (C)"
- note removed: "4. Speaker: simple = piezo direct to GP15+GND. Louder = NPN transistor amplifier"
- note removed: "5. Total GPIO used: 16 of 26. Free: GP7, GP17-22, GP26-28 (10 pins)"
- note removed: "6. 3V3(OUT) max 300mA — total draw ~120mA with all peripherals active"
- note removed: "7. GPS needs clear sky view for satellite fix — first fix takes 1-5 minutes"
- note removed: "BUSY ──→ GP13 [Pin 17]"
- note removed: "CENTER/SET ──→ GP6 [Pin 9] (internal pull-up)"
- note removed: "CLK ──→ GP10 (SPI1 SCK) [Pin 14]"
- note removed: "COM/GND ──→ GND [Pin 8]"
- note removed: "CS ──→ GP9 (SPI1 CSn) [Pin 12]"
- note removed: "DC ──→ GP8 [Pin 11]"
- note removed: "DIN ──→ GP11 (SPI1 TX) [Pin 15]"
- note removed: "DOLLATEK 5-WAY JOYSTICK (GPIO, Active LOW)"
- note removed: "DOWN ──→ GP3 [Pin 5] (internal pull-up)"
- note removed: "ECHO ──→ [1KΩ]──┬──→ GP16 [Pin 21] ⚠ DIVIDER REQUIRED"
- note removed: "GND [13]"
- note removed: "GND [18]"
- note removed: "GND [23] — HC-SR04 GND + Speaker GND"
- note removed: "GND [38] — e-Paper GND"
- note removed: "GND [3] — GPS GND"
- note removed: "GND [8] — Joystick COM/GND"
- note removed: "GND ──→ Emitter (E)"
- note removed: "GND ──→ GND [Pin 23]"
- note removed: "GND ──→ GND [Pin 38]"
- note removed: "GP0 [1] — UART0 TX → GPS RX"
- note removed: "GP1 [2] — UART0 RX ← GPS TX"
- note removed: "GP10 [14] — e-Paper CLK (SPI1 SCK)"
- note removed: "GP11 [15] — e-Paper DIN (SPI1 TX)"
- note removed: "GP12 [16] — e-Paper RST"
- note removed: "GP13 [17] — e-Paper BUSY"
- note removed: "GP14 [19] — HC-SR04 TRIG"
- note removed: "GP15 [20] — Speaker PWM"
- note removed: "GP15 ──[1KΩ R3]──→ Base (B)"
- note removed: "GP16 [21] — HC-SR04 ECHO (via 1K+2K divider)"
- note removed: "GP2 [4] — Joystick UP (pull-up, active LOW)"
- note removed: "GP3 [5] — Joystick DOWN"
- note removed: "GP4 [6] — Joystick LEFT"
- note removed: "GP5 [7] — Joystick RIGHT"
- note removed: "GP6 [9] — Joystick CENTER/SELECT"
- note removed: "GP7 [10] — FREE"
- note removed: "GP8 [11] — e-Paper DC"
- note removed: "GP9 [12] — e-Paper CS (SPI1 CSn)"
- note removed: "GPS GND ──→ GND [Pin 3]"
- note removed: "GPS RX ←── GP0 (UART0 TX) [Pin 1] ← CROSSOVER"
- note removed: "GPS TX ──→ GP1 (UART0 RX) [Pin 2] ← CROSSOVER"
- note removed: "GPS VCC ──→ 3V3(OUT) [Pin 36]"
- note removed: "GY-NEO6MV2 GPS MODULE (UART0, 9600 baud)"
- note removed: "HC-SR04 ECHO VOLTAGE DIVIDER (5V → 3.3V)"
- note removed: "HC-SR04 ECHO ──[1KΩ R1]──┬──→ GP16 (Pin 21)"
- note removed: "HC-SR04 ULTRASONIC SENSOR (5V, voltage divider on ECHO)"
- note removed: "LEFT ──→ GP4 [Pin 6] (internal pull-up)"
- note removed: "RASPBERRY PI PICO WH"
- note removed: "RIGHT ──→ GP5 [Pin 7] (internal pull-up)"
- note removed: "RST ──→ GP12 [Pin 16]"
- note removed: "SPEAKER CIRCUIT (PWM + NPN Transistor)"
- note removed: "Simple option: GP15 ──→ Piezo(+), GND ──→ Piezo(-)"
- note removed: "TRIG ──→ GP14 [Pin 19] (3.3V output is sufficient)"
- note removed: "Transistor: 2N2222, BC547, or BC817 (NPN)"
- note removed: "UP ──→ GP2 [Pin 4] (internal pull-up)"
- note removed: "VBUS [40] — HC-SR04 VCC (5V)"
- note removed: "VCC ──→ 3V3(OUT) [Pin 36]"
- note removed: "VCC ──→ VBUS (5V) [Pin 40] ⚠ MUST BE 5V"
- note removed: "VSYS [39] — (Battery future)"
- note removed: "Vout = 5V × 2K/(1K+2K) = 3.33V ✓"
- note removed: "WAVESHARE 2.13" e-PAPER V3 (SPI1, 4MHz)"
- note removed: "[2KΩ R2]"
- note removed: "[2KΩ]──→ GND"
- note removed: "│"
- title: Dilder Breadboard Test Bench -> Dilder Breadboard Test Bench — Full Wiring Reference
