File: hardware-design/joystick-pcb/joystick-pcb.kicad_pcb (KiCad board)
At the start: 2 copper layers, 20 x 20 mm, 6 parts, among them J1 Wire_Pads, SW1 SKRHABE010

Commit message: slight adjustments to pcb board for legibility
Changed lines of the file:
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@@
 		)
 		(property "Value" "SKRHABE010"
-			(at 0 5.5 0)
+			(at -8.15 0 90)
 			(layer "F.Fab")
 			(effects
@@
 	)
 	(gr_text "UP"
-		(at 105.5 115.7 0)
+		(at 105.5 119 0)
 		(layer "F.SilkS")
 		(effects
@@
 	)
 	(gr_text "DN"
-		(at 107.3 115.7 0)
+		(at 107.3 119 0)
 		(layer "F.SilkS")
 		(effects
@@
 	)
 	(gr_text "LT"
-		(at 109.1 115.7 0)
+		(at 109 119 0)
 		(layer "F.SilkS")
 		(effects
@@
 	)
 	(gr_text "RT"
-		(at 110.9 115.7 0)
+		(at 111 119 0)
 		(layer "F.SilkS")
 		(effects
@@
 	)
 	(gr_text "CT"
-		(at 112.7 115.7 0)
+		(at 112.7 119 0)
 		(layer "F.SilkS")
 		(effects
@@
 	)
 	(gr_text "GND"
-		(at 114.5 115.7 0)
-		(layer "F.SilkS")
-		(effects
+		(at 115 119 0)
+		(layer "F.SilkS")
+		(effects
